File: hardware/irblaster.kicad_sch (KiCad schematic)
At the start: 0 parts

Commit message: placed components initially
Parts:
- added U1: CH32V003FxPx, Package_SO:TSSOP-20_4.4x6.5mm_P0.65mm, symbol MCU_WCH_CH32V0:CH32V003FxPx
- added U2: TLV70033_SOT23-5, Package_TO_SOT_SMD:SOT-23-5, symbol Regulator_Linear:TLV70033_SOT23-5
- added U3: TP4057, Package_TO_SOT_SMD:TSOT-23-6, symbol Battery_Management:TP4057
